File: design/TX_Hand/TX_Hand.kicad_pcb (KiCad board)
At the start: 2 copper layers, 71.2 x 53.8 mm, 32 parts, among them J1 V_Battery, J2 STLINK, J3 UART, J8 PINHD_1x3_Male, SW1 SW_DPST_x2, SW2 SW_DPST_x2, U1 STM32F103C8Tx, U2 AMS1117-3.3, U4 NRF24L01_Breakout, U5 GY-521, X1 Crystal

Commit message: feat: TX_HAND autoroute try 10-10
Parts:
- moved U2 0.25 mm to (137.4, 95.0)
Routing:
- net VCC: track 163.2 -> 247.9 mm
- net GND: track 221.3 -> 173.8 mm
- net CSN: track 0.00 -> 20.7 mm
- net IRQ: track 0.00 -> 19.9 mm
- net CE: track 0.00 -> 19.0 mm
- net MISO: track 0.00 -> 14.9 mm
- net SCK: track 15.4 -> 25.1 mm
- net SDA: track 23.5 -> 14.9 mm
- net TX: track 13.6 -> 21.5 mm
- net SW_LUZ: track 19.5 -> 15.2 mm
- net ADC2: track 70.6 -> 66.5 mm
- net RX: track 14.9 -> 18.5 mm
- net SCL: track 16.9 -> 20.1 mm
- net RED: track 10.8 -> 9.47 mm
- net Net-(U1-PB2): track 6.31 -> 5.28 mm
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
Commit message: fix: merge changes of Ale
Parts:
- added C10: 10uF, Capacitor_SMD:C_0805_2012Metric_Pad1.18x1.45mm_HandSolder, F.Cu at (180.9, 100.8)
- added C11: 22uF, Capacitor_SMD:C_0805_2012Metric_Pad1.18x1.45mm_HandSolder, F.Cu at (180.9, 103.8)
- added U3: AMS1117-3.3, Package_TO_SOT_SMD:SOT-223-3_TabPin2, F.Cu at (183.5, 95.2)
- J8: value PINHD_1x3_Male -> ADC
Connections:
- C7 pad 2: GND -> Net-(C7-Pad2)
- C8 pad 2: GND -> Net-(C7-Pad2)
- U4 pad 1: unconnected-(U4-GND-Pad1) -> GND
- U4 pad 2: VCC -> VCC_RF
