File: design/TX_Hand/TX_Hand.kicad_sch (KiCad schematic)
At the start: 32 parts, among them J1 V_Battery, J2 STLINK, J3 UART, J8 PINHD_1x3_Male, SW1 SW_DPST_x2, SW2 SW_DPST_x2, U1 STM32F103C8Tx, U2 AMS1117-3.3, U4 NRF24L01_Breakout, U5 GY-521, X1 Crystal

Commit message: chore: minor fixes
Parts:
- U5: footprint GY-521:MODULE_GY-521 -> GY-521 (1):MODULE_GY-521
Changed lines of the file:
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@@
 			)
 		)
-		(property "Footprint" "GY-521:MODULE_GY-521"
+		(property "Footprint" "GY-521 (1):MODULE_GY-521"
 			(at 40.386 173.228 0)
 			(hide yes)

Commit message: fix: merge changes of Ale
Parts:
- added C10: 10uF, Capacitor_SMD:C_0805_2012Metric_Pad1.18x1.45mm_HandSolder, symbol Device:C_Polarized
- added C11: 22uF, Capacitor_SMD:C_0805_2012Metric_Pad1.18x1.45mm_HandSolder, symbol Device:C_Polarized
- added U3: AMS1117-3.3, Package_TO_SOT_SMD:SOT-223-3_TabPin2, symbol Regulator_Linear:AMS1117-3.3
- J8: value PINHD_1x3_Male -> ADC
Connections:
- net GND: now also U4.1 (GND), U3.1 (GND); no longer C7.2, C8.2
- net VCC: no longer U4.2 (VCC)
- net VIN: now also C10.1, U3.3 (VI)
- new net: C10.2, C11.2
- new net: C7.2, C8.2
- new net VCC_RF: C11.1, U3.2 (VO), U4.2 (VCC)
Other:
- moved on the sheet: C7, C8, D1, D2, D3, J1, J3, J8, R5, R6, R8, R9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
